File: PCB/pcb.sch (KiCad schematic (older format))
At the start: 220 parts, among them J1 USB_C_Receptacle_USB2.0, SW1 SW_Push, U1 AT90USB1286-AU, Y1 Crystal_GND24_Small

Commit message: Changed Switches to have no LED
+Wired left arrow
Parts:
- removed MX*1, MX+1, MX+2, MX,1, MX,2, MX-1, MX-2, MX.1, MX/1, MX0, MX1, MX10, MX11, MX13, MX14, MX15, MX16, MX17, MX2, MX3, MX4, MX5, MX6, MX7, MX8, MX9, MX^1, MXa1, MXalt1, MXaltgr1, MXb1, MXback1, MXc1, MXcaps1, MXctrl1, MXd1, MXdel1, MXdown1, MXdruck1, MXe1, MXenter1, MXesc1, MXf0, MXf1, MXf10, MXf11, MXf12, MXf2, MXf3, MXf4, MXf5, MXf6, MXf7, MXf8, MXf9, MXfn1, MXg1, MXh1, MXi1, MXinsert1, MXj1, MXk1, MXl1, MXleer1, MXleft1, MXm1, MXn1, MXnum0, MXnum1, MXnum2, MXnum3, MXnum4, MXnum5, MXnum6, MXnum7, MXnum8, MXnum9, MXnumlock1, MXo1, MXp1, MXpgdn1, MXpgup1, MXq1, MXr1, MXright1, MXs1, MXshift1, MXshift2, MXt1, MXtab1, MXu1, MXup1, MXv1, MXv2, MXw1, MXwin1, MXwin2, MXx1, MXy1, MXz1: MX-LED, MX_Alps_Hybrid:MX-1U, symbol MX_Alps_Hybrid:MX-LED
- added MX? (x100): MX-NoLED, symbol MX_Alps_Hybrid:MX-NoLED
Connections:
- net COL0: now also MX?.1 (COL), MX?.1 (COL), MX?.1 (COL), MX?.1 (COL), MX?.1 (COL), MX?.1 (COL)
- net COL1: now also MX?.1 (COL), MX?.1 (COL), MX?.1 (COL), MX?.1 (COL), MX?.1 (COL)
- net COL10: now also MX?.1 (COL), MX?.1 (COL), MX?.1 (COL), MX?.1 (COL), MX?.1 (COL), MX?.1 (COL)
- net COL11: now also MX?.1 (COL), MX?.1 (COL), MX?.1 (COL), MX?.1 (COL), MX?.1 (COL), MX?.1 (COL)
- net COL12: now also MX?.1 (COL), MX?.1 (COL), MX?.1 (COL), MX?.1 (COL), MX?.1 (COL), MX?.1 (COL)
- net COL13: now also MX?.1 (COL), MX?.1 (COL), MX?.1 (COL), MX?.1 (COL), MX?.1 (COL)
- net COL14: now also MX?.1 (COL), MX?.1 (COL), MX?.1 (COL), MX?.1 (COL), MX?.1 (COL), MX?.1 (COL)
- net COL15: now also MX?.1 (COL), MX?.1 (COL), MX?.1 (COL), MX?.1 (COL), MX?.1 (COL)
- net COL16: now also MX?.1 (COL), MX?.1 (COL), MX?.1 (COL), MX?.1 (COL), MX?.1 (COL), MX?.1 (COL)
- net COL17: now also MX?.1 (COL), MX?.1 (COL), MX?.1 (COL)
- net COL2: now also MX?.1 (COL), MX?.1 (COL), MX?.1 (COL), MX?.1 (COL), MX?.1 (COL), MX?.1 (COL)
- net COL3: now also MX?.1 (COL), MX?.1 (COL), MX?.1 (COL), MX?.1 (COL), MX?.1 (COL)
- net COL4: now also MX?.1 (COL), MX?.1 (COL), MX?.1 (COL), MX?.1 (COL), MX?.1 (COL)
- net COL5: now also MX?.1 (COL), MX?.1 (COL), MX?.1 (COL), MX?.1 (COL), MX?.1 (COL), MX?.1 (COL)
- net COL6: now also MX?.1 (COL), MX?.1 (COL), MX?.1 (COL), MX?.1 (COL), MX?.1 (COL), MX?.1 (COL)
- net COL7: now also MX?.1 (COL), MX?.1 (COL), MX?.1 (COL), MX?.1 (COL), MX?.1 (COL), MX?.1 (COL)
- net COL8: now also MX?.1 (COL), MX?.1 (COL), MX?.1 (COL), MX?.1 (COL), MX?.1 (COL), MX?.1 (COL)
- net COL9: now also MX?.1 (COL), MX?.1 (COL), MX?.1 (COL), MX?.1 (COL), MX?.1 (COL), MX?.1 (COL)
- net at D2.2 (A): now also MX?.2 (ROW)
- net at D7.2 (A): now also MX?.2 (ROW)
- net at D3.2 (A): now also MX?.2 (ROW)
- net at D8.2 (A): now also MX?.2 (ROW)
- net at D1.2 (A): now also MX?.2 (ROW)
- net at D4.2 (A): now also MX?.2 (ROW)
- net at D5.2 (A): now also MX?.2 (ROW)
- net at D6.2 (A): now also MX?.2 (ROW)
- net at D9.2 (A): now also MX?.2 (ROW)
- net at D10.2 (A): now also MX?.2 (ROW)
- net at D11.2 (A): now also MX?.2 (ROW)
- net at D13.2 (A): now also MX?.2 (ROW)
- net at D19.2 (A): now also MX?.2 (ROW)
- net at D14.2 (A): now also MX?.2 (ROW)
- net at D20.2 (A): now also MX?.2 (ROW)
- net at D15.2 (A): now also MX?.2 (ROW)
- net at D16.2 (A): now also MX?.2 (ROW)
- net at D17.2 (A): now also MX?.2 (ROW)
- net at D21.2 (A): now also MX?.2 (ROW)
- net at D22.2 (A): now also MX?.2 (ROW)
- net at D24.2 (A): now also MX?.2 (ROW)
- net at D29.2 (A): now also MX?.2 (ROW)
- net at D25.2 (A): now also MX?.2 (ROW)
- net at D30.2 (A): now also MX?.2 (ROW)
- net at D26.2 (A): now also MX?.2 (ROW)
- net at D27.2 (A): now also MX?.2 (ROW)
- net at D31.2 (A): now also MX?.2 (ROW)
- net at D32.2 (A): now also MX?.2 (ROW)
- net at D34.2 (A): now also MX?.2 (ROW)
- net at D40.2 (A): now also MX?.2 (ROW)
- net at D35.2 (A): now also MX?.2 (ROW)
- net at D41.2 (A): now also MX?.2 (ROW)
- net at D36.2 (A): now also MX?.2 (ROW)
- net at D37.2 (A): now also MX?.2 (ROW)
- net at D42.2 (A): now also MX?.2 (ROW)
- net at D43.2 (A): now also MX?.2 (ROW)
- net at D45.2 (A): now also MX?.2 (ROW)
- net at D50.2 (A): now also MX?.2 (ROW)
- net at D46.2 (A): now also MX?.2 (ROW)
- net at D51.2 (A): now also MX?.2 (ROW)
- net at D47.2 (A): now also MX?.2 (ROW)
- net at D48.2 (A): now also MX?.2 (ROW)
- net at D52.2 (A): now also MX?.2 (ROW)
- net at D53.2 (A): now also MX?.2 (ROW)
- net at D55.2 (A): now also MX?.2 (ROW)
- net at D61.2 (A): now also MX?.2 (ROW)
- net at D56.2 (A): now also MX?.2 (ROW)
- net at D62.2 (A): now also MX?.2 (ROW)
- net at D57.2 (A): now also MX?.2 (ROW)
- net at D58.2 (A): now also MX?.2 (ROW)
- net at D63.2 (A): now also MX?.2 (ROW)
- net at D64.2 (A): now also MX?.2 (ROW)
- net at D67.2 (A): now also MX?.2 (ROW)
- net at D73.2 (A): now also MX?.2 (ROW)
- net at D68.2 (A): now also MX?.2 (ROW)
- net at D74.2 (A): now also MX?.2 (ROW)
- net at D69.2 (A): now also MX?.2 (ROW)
- net at D70.2 (A): now also MX?.2 (ROW)
- net at D78.2 (A): now also MX?.2 (ROW)
- net at D75.2 (A): now also MX?.2 (ROW)
- net at D76.2 (A): now also MX?.2 (ROW)
- net at D77.2 (A): now also MX?.2 (ROW)
- net at D12.2 (A): now also MX?.2 (ROW)
- net at D18.2 (A): now also MX?.2 (ROW)
- net at D23.2 (A): now also MX?.2 (ROW)
- net at D28.2 (A): now also MX?.2 (ROW)
- net at D33.2 (A): now also MX?.2 (ROW)
- net at D39.2 (A): now also MX?.2 (ROW)
- net at D44.2 (A): now also MX?.2 (ROW)
- net at D49.2 (A): now also MX?.2 (ROW)
- net at D54.2 (A): now also MX?.2 (ROW)
- net at D60.2 (A): now also MX?.2 (ROW)
- net at D66.2 (A): now also MX?.2 (ROW)
- net at D72.2 (A): now also MX?.2 (ROW)
- net at D38.2 (A): now also MX?.2 (ROW)
- net at D59.2 (A): now also MX?.2 (ROW)
- net at D65.2 (A): now also MX?.2 (ROW)
- net at D71.2 (A): now also MX?.2 (ROW)
- net at D80.2 (A): now also MX?.2 (ROW)
- net at D81.2 (A): now also MX?.2 (ROW)
- net at D82.2 (A): now also MX?.2 (ROW)
- net at D83.2 (A): now also MX?.2 (ROW)
- net at D79.2 (A): now also MX?.2 (ROW)
- net at D85.2 (A): now also MX?.2 (ROW)
- net at D86.2 (A): now also MX?.2 (ROW)
- net at D87.2 (A): now also MX?.2 (ROW)
- net at D88.2 (A): now also MX?.2 (ROW)
- net at D90.2 (A): now also MX?.2 (ROW)
- net at D95.2 (A): now also MX?.2 (ROW)
- net at D91.2 (A): now also MX?.2 (ROW)
- net at D96.2 (A): now also MX?.2 (ROW)
- net at D92.2 (A): now also MX?.2 (ROW)
- net at D97.2 (A): now also MX?.2 (ROW)
- net at D93.2 (A): now also MX?.2 (ROW)
- net at D99.2 (A): now also MX?.2 (ROW)
- net at D100.2 (A): now also MX?.2 (ROW)
- net at D84.2 (A): now also MX?.2 (ROW)
- net at D89.2 (A): now also MX?.2 (ROW)
- net at D94.2 (A): now also MX?.2 (ROW)
- net at D98.2 (A): now also MX?.2 (ROW)
