File: PCB/pcb.kicad_pcb (KiCad board)
At the start: 2 copper layers, 403.2 x 127 mm, 324 parts, among them J1 USB_C_Receptacle_USB2.0, SW1 SW_Push, U1 AT90USB1286-AU, Y1 Crystal_GND24_Small

Commit message: LED Shenanigans
Parts:
- D101, D102, D103, D104, D105, D106, D107, D108, D109, D110, D111, D112, D113, D114, D115, D116, D117, D118, D119, D120, D121, D122, D123, D124, D125, D126, D127, D128, D129, D130, D131, D132, D133, D134, D135, D136, D137, D138, D139, D140, D141, D142, D143, D144, D145, D146, D147, D148, D149, D150, D151, D152, D153, D154, D155, D156, D157, D158, D159, D160, D161, D162, D163, D164, D165, D166, D167, D168, D169, D170, D171, D172, D173, D174, D175, D176, D177, D178, D179, D180, D181, D182, D183, D184, D185, D186, D187, D188, D189, D190, D191, D192, D193, D194, D195, D196, D197, D198, D199, D200: footprint led:SK6812MINI_3.5x3.7mm_SMD-Back -> led:SK6812MINI_3.5x3.7mm_SMD-Flipped-Back
- renumbered Cre to C3
Connections:
- D102 pad 1: Net-(D102-Pad1) -> unconnected-(D102-Pad1)
- D102 pad 3: RGBDOUT0 -> Net-(D101-Pad1)
- D103 pad 2: GND -> unconnected-(D103-Pad2)
- D103 pad 3: RGBDOUT1 -> unconnected-(D103-Pad3)
- D103 pad 4: +5V -> unconnected-(D103-Pad4)
- D104 pad 1: Net-(D104-Pad1) -> unconnected-(D104-Pad1)
- D104 pad 3: RGBDOUT2 -> Net-(D103-Pad1)
- D105 pad 2: GND -> unconnected-(D105-Pad2)
- D105 pad 3: RGBDOUT3 -> unconnected-(D105-Pad3)
- D105 pad 4: +5V -> unconnected-(D105-Pad4)
- D106 pad 3: RGBDOUT4 -> Net-(D105-Pad1)
- D107 pad 3: RGBDOUT5 -> Net-(D106-Pad1)
- D108 pad 3: RGBDOUT6 -> Net-(D107-Pad1)
- D109 pad 3: RGBDOUT7 -> Net-(D108-Pad1)
- D110 pad 1: Net-(D110-Pad1) -> RGBDOUT0
- D110 pad 3: RGBDOUT8 -> Net-(D109-Pad1)
- D111 pad 3: Net-(D101-Pad1) -> RGBDOUT0
- D112 pad 1: Net-(D112-Pad1) -> Net-(D113-Pad3)
- D112 pad 3: Net-(D102-Pad1) -> Net-(D111-Pad1)
- D113 pad 3: Net-(D103-Pad1) -> Net-(D113-Pad3)
- D114 pad 3: Net-(D104-Pad1) -> Net-(D113-Pad1)
- D115 pad 1: Net-(D115-Pad1) -> unconnected-(D115-Pad1)
- D115 pad 3: Net-(D105-Pad1) -> Net-(D114-Pad1)
- D116 pad 2: GND -> unconnected-(D116-Pad2)
- D116 pad 3: Net-(D106-Pad1) -> unconnected-(D116-Pad3)
- D116 pad 4: +5V -> unconnected-(D116-Pad4)
- D117 pad 3: Net-(D107-Pad1) -> Net-(D116-Pad1)
- D118 pad 3: Net-(D108-Pad1) -> Net-(D117-Pad1)
- D119 pad 3: Net-(D109-Pad1) -> Net-(D118-Pad1)
- D120 pad 1: Net-(D120-Pad1) -> RGBDOUT1
- D120 pad 3: Net-(D110-Pad1) -> Net-(D119-Pad1)
- D121 pad 3: Net-(D111-Pad1) -> RGBDOUT1
- D122 pad 1: Net-(D122-Pad1) -> unconnected-(D122-Pad1)
- D122 pad 2: GND -> unconnected-(D122-Pad2)
- D122 pad 3: Net-(D112-Pad1) -> Net-(D121-Pad1)
- D122 pad 4: +5V -> unconnected-(D122-Pad4)
- D123 pad 3: Net-(D113-Pad1) -> unconnected-(D123-Pad3)
- D124 pad 3: Net-(D114-Pad1) -> Net-(D123-Pad1)
- D125 pad 3: Net-(D115-Pad1) -> Net-(D124-Pad1)
- D126 pad 3: Net-(D116-Pad1) -> Net-(D125-Pad1)
- D127 pad 3: Net-(D117-Pad1) -> Net-(D126-Pad1)
- D128 pad 1: Net-(D128-Pad1) -> Net-(D129-Pad3)
- D128 pad 3: Net-(D118-Pad1) -> Net-(D127-Pad1)
- D129 pad 3: Net-(D119-Pad1) -> Net-(D129-Pad3)
- D130 pad 1: Net-(D130-Pad1) -> RGBDOUT2
- D130 pad 3: Net-(D120-Pad1) -> Net-(D129-Pad1)
- D131 pad 3: Net-(D121-Pad1) -> RGBDOUT2
- D132 pad 3: Net-(D122-Pad1) -> Net-(D131-Pad1)
- D133 pad 3: Net-(D123-Pad1) -> Net-(D132-Pad1)
- D134 pad 3: Net-(D124-Pad1) -> Net-(D133-Pad1)
- D135 pad 3: Net-(D125-Pad1) -> Net-(D134-Pad1)
- D136 pad 3: Net-(D126-Pad1) -> Net-(D135-Pad1)
- D137 pad 3: Net-(D127-Pad1) -> Net-(D136-Pad1)
- D138 pad 1: Net-(D138-Pad1) -> Net-(D139-Pad3)
- D138 pad 3: Net-(D128-Pad1) -> Net-(D137-Pad1)
- D139 pad 1: Net-(D139-Pad1) -> unconnected-(D139-Pad1)
- D139 pad 2: GND -> unconnected-(D139-Pad2)
- D139 pad 3: Net-(D129-Pad1) -> Net-(D139-Pad3)
- D139 pad 4: +5V -> unconnected-(D139-Pad4)
- D140 pad 1: Net-(D140-Pad1) -> RGBDOUT3
- D140 pad 3: Net-(D130-Pad1) -> unconnected-(D140-Pad3)
- D141 pad 1: Net-(D141-Pad1) -> Net-(D142-Pad3)
- D141 pad 3: Net-(D131-Pad1) -> RGBDOUT3
- D142 pad 3: Net-(D132-Pad1) -> Net-(D142-Pad3)
- D143 pad 1: Net-(D143-Pad1) -> Net-(D144-Pad3)
- D143 pad 3: Net-(D133-Pad1) -> Net-(D142-Pad1)
- D144 pad 3: Net-(D134-Pad1) -> Net-(D144-Pad3)
- D145 pad 1: Net-(D145-Pad1) -> Net-(D146-Pad3)
- D145 pad 3: Net-(D135-Pad1) -> Net-(D144-Pad1)
- D146 pad 3: Net-(D136-Pad1) -> Net-(D146-Pad3)
- D147 pad 3: Net-(D137-Pad1) -> Net-(D146-Pad1)
- D148 pad 3: Net-(D138-Pad1) -> Net-(D147-Pad1)
- D149 pad 1: Net-(D149-Pad1) -> Net-(D150-Pad3)
- D149 pad 3: Net-(D139-Pad1) -> Net-(D148-Pad1)
- D150 pad 1: Net-(D150-Pad1) -> RGBDOUT4
- D150 pad 3: Net-(D140-Pad1) -> Net-(D150-Pad3)
- D151 pad 1: Net-(D151-Pad1) -> Net-(D152-Pad3)
- D151 pad 3: Net-(D141-Pad1) -> RGBDOUT4
- D152 pad 1: Net-(D152-Pad1) -> Net-(D153-Pad3)
- D152 pad 3: Net-(D142-Pad1) -> Net-(D152-Pad3)
- D153 pad 3: Net-(D143-Pad1) -> Net-(D153-Pad3)
- D154 pad 3: Net-(D144-Pad1) -> Net-(D153-Pad1)
- D155 pad 1: Net-(D155-Pad1) -> Net-(D156-Pad3)
- D155 pad 3: Net-(D145-Pad1) -> Net-(D154-Pad1)
- D156 pad 3: Net-(D146-Pad1) -> Net-(D156-Pad3)
- D157 pad 3: Net-(D147-Pad1) -> Net-(D156-Pad1)
- D158 pad 3: Net-(D148-Pad1) -> Net-(D157-Pad1)
- D159 pad 3: Net-(D149-Pad1) -> Net-(D158-Pad1)
- D160 pad 1: Net-(D160-Pad1) -> RGBDOUT5
- D160 pad 3: Net-(D150-Pad1) -> Net-(D159-Pad1)
- D161 pad 3: Net-(D151-Pad1) -> RGBDOUT5
- D162 pad 1: Net-(D162-Pad1) -> Net-(D163-Pad3)
- D162 pad 3: Net-(D152-Pad1) -> Net-(D161-Pad1)
- D163 pad 3: Net-(D153-Pad1) -> Net-(D163-Pad3)
- D164 pad 3: Net-(D154-Pad1) -> Net-(D163-Pad1)
- D165 pad 3: Net-(D155-Pad1) -> Net-(D164-Pad1)
- D166 pad 1: Net-(D166-Pad1) -> Net-(D167-Pad3)
- D166 pad 3: Net-(D156-Pad1) -> Net-(D165-Pad1)
- D167 pad 3: Net-(D157-Pad1) -> Net-(D167-Pad3)
- D168 pad 3: Net-(D158-Pad1) -> Net-(D167-Pad1)
- D169 pad 3: Net-(D159-Pad1) -> Net-(D168-Pad1)
- D170 pad 1: Net-(D170-Pad1) -> RGBDOUT6
- D170 pad 3: Net-(D160-Pad1) -> Net-(D169-Pad1)
- D171 pad 3: Net-(D161-Pad1) -> RGBDOUT6
- D172 pad 3: Net-(D162-Pad1) -> Net-(D171-Pad1)
- D173 pad 3: Net-(D163-Pad1) -> Net-(D172-Pad1)
- D174 pad 3: Net-(D164-Pad1) -> Net-(D173-Pad1)
- D175 pad 3: Net-(D165-Pad1) -> Net-(D174-Pad1)
- D176 pad 1: Net-(D176-Pad1) -> Net-(D177-Pad3)
- D176 pad 3: Net-(D166-Pad1) -> Net-(D175-Pad1)
- D177 pad 3: Net-(D167-Pad1) -> Net-(D177-Pad3)
- D178 pad 3: Net-(D168-Pad1) -> Net-(D177-Pad1)
- D179 pad 1: Net-(D179-Pad1) -> Net-(D180-Pad3)
- D179 pad 3: Net-(D169-Pad1) -> Net-(D178-Pad1)
- D180 pad 1: Net-(D180-Pad1) -> RGBDOUT7
- D180 pad 3: Net-(D170-Pad1) -> Net-(D180-Pad3)
- D181 pad 3: Net-(D171-Pad1) -> RGBDOUT7
- D182 pad 3: Net-(D172-Pad1) -> Net-(D181-Pad1)
- D183 pad 3: Net-(D173-Pad1) -> Net-(D182-Pad1)
- D184 pad 3: Net-(D174-Pad1) -> Net-(D183-Pad1)
- D185 pad 3: Net-(D175-Pad1) -> Net-(D184-Pad1)
- D186 pad 3: Net-(D176-Pad1) -> Net-(D185-Pad1)
- D187 pad 1: Net-(D187-Pad1) -> Net-(D188-Pad3)
- D187 pad 3: Net-(D177-Pad1) -> Net-(D186-Pad1)
- D188 pad 1: Net-(D188-Pad1) -> Net-(D189-Pad3)
- D188 pad 3: Net-(D178-Pad1) -> Net-(D188-Pad3)
- D189 pad 3: Net-(D179-Pad1) -> Net-(D189-Pad3)
- D190 pad 1: Net-(D190-Pad1) -> RGBDOUT8
- D190 pad 3: Net-(D180-Pad1) -> Net-(D189-Pad1)
- D191 pad 1: RGBDOUT0 -> Net-(D191-Pad1)
- D191 pad 3: Net-(D181-Pad1) -> RGBDOUT8
- D192 pad 1: RGBDOUT1 -> Net-(D192-Pad1)
- D192 pad 3: Net-(D182-Pad1) -> Net-(D191-Pad1)
- D193 pad 1: RGBDOUT2 -> Net-(D193-Pad1)
- D193 pad 3: Net-(D183-Pad1) -> Net-(D192-Pad1)
- D194 pad 1: RGBDOUT3 -> Net-(D194-Pad1)
- D194 pad 3: Net-(D184-Pad1) -> Net-(D193-Pad1)
- D195 pad 1: RGBDOUT4 -> Net-(D195-Pad1)
- D195 pad 3: Net-(D185-Pad1) -> Net-(D194-Pad1)
- D196 pad 1: RGBDOUT5 -> Net-(D196-Pad1)
- D196 pad 3: Net-(D186-Pad1) -> Net-(D195-Pad1)
- D197 pad 1: RGBDOUT6 -> Net-(D198-Pad3)
- D197 pad 3: Net-(D187-Pad1) -> Net-(D196-Pad1)
- D198 pad 1: RGBDOUT7 -> Net-(D199-Pad3)
- D198 pad 3: Net-(D188-Pad1) -> Net-(D198-Pad3)
- D199 pad 1: RGBDOUT8 -> Net-(D200-Pad3)
- D199 pad 3: Net-(D189-Pad1) -> Net-(D199-Pad3)
- D200 pad 3: Net-(D190-Pad1) -> Net-(D200-Pad3)

Commit message: LED Data Buses finished
Connections:
- D102 pad 1: unconnected-(D102-Pad1) -> Net-(D102-Pad1)
- D103 pad 2: unconnected-(D103-Pad2) -> GND
- D103 pad 3: unconnected-(D103-Pad3) -> Net-(D102-Pad1)
- D103 pad 4: unconnected-(D103-Pad4) -> +5V
- D104 pad 1: unconnected-(D104-Pad1) -> Net-(D105-Pad3)
- D105 pad 2: unconnected-(D105-Pad2) -> GND
- D105 pad 3: unconnected-(D105-Pad3) -> Net-(D105-Pad3)
- D105 pad 4: unconnected-(D105-Pad4) -> +5V
- D115 pad 1: unconnected-(D115-Pad1) -> Net-(D115-Pad1)
- D116 pad 2: unconnected-(D116-Pad2) -> GND
- D116 pad 3: unconnected-(D116-Pad3) -> Net-(D115-Pad1)
- D116 pad 4: unconnected-(D116-Pad4) -> +5V
- D122 pad 1: unconnected-(D122-Pad1) -> Net-(D123-Pad3)
- D122 pad 2: unconnected-(D122-Pad2) -> GND
- D122 pad 4: unconnected-(D122-Pad4) -> +5V
- D123 pad 3: unconnected-(D123-Pad3) -> Net-(D123-Pad3)
- D139 pad 1: unconnected-(D139-Pad1) -> Net-(D140-Pad3)
- D139 pad 2: unconnected-(D139-Pad2) -> GND
- D139 pad 4: unconnected-(D139-Pad4) -> +5V
- D140 pad 3: unconnected-(D140-Pad3) -> Net-(D140-Pad3)
Routing:
- net Net-(D159-Pad1): track 0.00 -> 155.4 mm, vias 0 -> 2
- net Net-(D171-Pad1): track 0.00 -> 139.5 mm, vias 0 -> 2
- net Net-(D165-Pad1): track 0.00 -> 133.2 mm, vias 0 -> 4
- net Net-(D139-Pad3): track 0.00 -> 130.9 mm, vias 0 -> 2
- net Net-(D178-Pad1): track 0.00 -> 122.1 mm, vias 0 -> 2
- net Net-(D117-Pad1): track 0.00 -> 120.6 mm, vias 0 -> 2
- net Net-(D153-Pad1): track 0.00 -> 117.1 mm, vias 0 -> 2
- net Net-(D111-Pad1): track 0.00 -> 114.2 mm, vias 0 -> 2
- net Net-(D148-Pad1): track 0.00 -> 107.6 mm, vias 0 -> 2
- net Net-(D144-Pad3): track 0.00 -> 106.2 mm, vias 0 -> 2
- net Net-(D132-Pad1): track 0.00 -> 105.9 mm, vias 0 -> 2
- net Net-(D123-Pad3): track 0.00 -> 100.1 mm, vias 0 -> 2
- net Net-(D127-Pad1): track 0.00 -> 98.2 mm, vias 0 -> 2
- net Net-(D193-Pad1): track 0.00 -> 97.8 mm, vias 0 -> 2
- net Net-(D189-Pad3): track 0.00 -> 90.5 mm, vias 0 -> 2
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
Commit message: Added LED Net
Connections:
- D101 pad 1: Net-(D101-Pad1) -> /LED
- D102 pad 1: Net-(D102-Pad1) -> /LED
- D102 pad 3: Net-(D101-Pad1) -> /LED
- D103 pad 1: Net-(D103-Pad1) -> /LED
- D103 pad 3: Net-(D102-Pad1) -> /LED
- D104 pad 1: Net-(D105-Pad3) -> /LED
- D104 pad 3: Net-(D103-Pad1) -> /LED
- D105 pad 1: Net-(D105-Pad1) -> /LED
- D105 pad 3: Net-(D105-Pad3) -> /LED
- D106 pad 1: Net-(D106-Pad1) -> /LED
- D106 pad 3: Net-(D105-Pad1) -> /LED
- D107 pad 1: Net-(D107-Pad1) -> /LED
- D107 pad 3: Net-(D106-Pad1) -> /LED
- D108 pad 1: Net-(D108-Pad1) -> /LED
- D108 pad 3: Net-(D107-Pad1) -> /LED
- D109 pad 1: Net-(D109-Pad1) -> /LED
- D109 pad 3: Net-(D108-Pad1) -> /LED
- D110 pad 1: RGBDOUT0 -> /LED
- D110 pad 3: Net-(D109-Pad1) -> /LED
- D111 pad 1: Net-(D111-Pad1) -> /LED
- D111 pad 3: RGBDOUT0 -> /LED
- D112 pad 1: Net-(D113-Pad3) -> /LED
- D112 pad 3: Net-(D111-Pad1) -> /LED
- D113 pad 1: Net-(D113-Pad1) -> /LED
- D113 pad 3: Net-(D113-Pad3) -> /LED
- D114 pad 1: Net-(D114-Pad1) -> /LED
- D114 pad 3: Net-(D113-Pad1) -> /LED
- D115 pad 1: Net-(D115-Pad1) -> /LED
- D115 pad 3: Net-(D114-Pad1) -> /LED
- D116 pad 1: Net-(D116-Pad1) -> /LED
- D116 pad 3: Net-(D115-Pad1) -> /LED
- D117 pad 1: Net-(D117-Pad1) -> /LED
- D117 pad 3: Net-(D116-Pad1) -> /LED
- D118 pad 1: Net-(D118-Pad1) -> /LED
- D118 pad 3: Net-(D117-Pad1) -> /LED
- D119 pad 1: Net-(D119-Pad1) -> /LED
- D119 pad 3: Net-(D118-Pad1) -> /LED
- D120 pad 1: RGBDOUT1 -> /LED
- D120 pad 3: Net-(D119-Pad1) -> /LED
- D121 pad 1: Net-(D121-Pad1) -> /LED
- D121 pad 3: RGBDOUT1 -> /LED
- D122 pad 1: Net-(D123-Pad3) -> /LED
- D122 pad 3: Net-(D121-Pad1) -> /LED
- D123 pad 1: Net-(D123-Pad1) -> /LED
- D123 pad 3: Net-(D123-Pad3) -> /LED
- D124 pad 1: Net-(D124-Pad1) -> /LED
- D124 pad 3: Net-(D123-Pad1) -> /LED
- D125 pad 1: Net-(D125-Pad1) -> /LED
- D125 pad 3: Net-(D124-Pad1) -> /LED
- D126 pad 1: Net-(D126-Pad1) -> /LED
- D126 pad 3: Net-(D125-Pad1) -> /LED
- D127 pad 1: Net-(D127-Pad1) -> /LED
- D127 pad 3: Net-(D126-Pad1) -> /LED
- D128 pad 1: Net-(D129-Pad3) -> /LED
- D128 pad 3: Net-(D127-Pad1) -> /LED
- D129 pad 1: Net-(D129-Pad1) -> /LED
- D129 pad 3: Net-(D129-Pad3) -> /LED
- D130 pad 1: RGBDOUT2 -> /LED
- D130 pad 3: Net-(D129-Pad1) -> /LED
- D131 pad 1: Net-(D131-Pad1) -> /LED
- D131 pad 3: RGBDOUT2 -> /LED
- D132 pad 1: Net-(D132-Pad1) -> /LED
- D132 pad 3: Net-(D131-Pad1) -> /LED
- D133 pad 1: Net-(D133-Pad1) -> /LED
- D133 pad 3: Net-(D132-Pad1) -> /LED
- D134 pad 1: Net-(D134-Pad1) -> /LED
- D134 pad 3: Net-(D133-Pad1) -> /LED
- D135 pad 1: Net-(D135-Pad1) -> /LED
- D135 pad 3: Net-(D134-Pad1) -> /LED
- D136 pad 1: Net-(D136-Pad1) -> /LED
- D136 pad 3: Net-(D135-Pad1) -> /LED
- D137 pad 1: Net-(D137-Pad1) -> /LED
- D137 pad 3: Net-(D136-Pad1) -> /LED
- D138 pad 1: Net-(D139-Pad3) -> /LED
- D138 pad 3: Net-(D137-Pad1) -> /LED
- D139 pad 1: Net-(D140-Pad3) -> /LED
- D139 pad 3: Net-(D139-Pad3) -> /LED
- D140 pad 1: RGBDOUT3 -> /LED
- D140 pad 3: Net-(D140-Pad3) -> /LED
- D141 pad 1: Net-(D142-Pad3) -> /LED
- D141 pad 3: RGBDOUT3 -> /LED
- D142 pad 1: Net-(D142-Pad1) -> /LED
- D142 pad 3: Net-(D142-Pad3) -> /LED
- D143 pad 1: Net-(D144-Pad3) -> /LED
- D143 pad 3: Net-(D142-Pad1) -> /LED
- D144 pad 1: Net-(D144-Pad1) -> /LED
- D144 pad 3: Net-(D144-Pad3) -> /LED
- D145 pad 1: Net-(D146-Pad3) -> /LED
- D145 pad 3: Net-(D144-Pad1) -> /LED
- D146 pad 1: Net-(D146-Pad1) -> /LED
- D146 pad 3: Net-(D146-Pad3) -> /LED
- D147 pad 1: Net-(D147-Pad1) -> /LED
- D147 pad 3: Net-(D146-Pad1) -> /LED
- D148 pad 1: Net-(D148-Pad1) -> /LED
- D148 pad 3: Net-(D147-Pad1) -> /LED
- D149 pad 1: Net-(D150-Pad3) -> /LED
- D149 pad 3: Net-(D148-Pad1) -> /LED
- D150 pad 1: RGBDOUT4 -> /LED
- D150 pad 3: Net-(D150-Pad3) -> /LED
- D151 pad 1: Net-(D152-Pad3) -> /LED
- D151 pad 3: RGBDOUT4 -> /LED
- D152 pad 1: Net-(D153-Pad3) -> /LED
- D152 pad 3: Net-(D152-Pad3) -> /LED
- D153 pad 1: Net-(D153-Pad1) -> /LED
- D153 pad 3: Net-(D153-Pad3) -> /LED
- D154 pad 1: Net-(D154-Pad1) -> /LED
- D154 pad 3: Net-(D153-Pad1) -> /LED
- D155 pad 1: Net-(D156-Pad3) -> /LED
- D155 pad 3: Net-(D154-Pad1) -> /LED
- D156 pad 1: Net-(D156-Pad1) -> /LED
- D156 pad 3: Net-(D156-Pad3) -> /LED
- D157 pad 1: Net-(D157-Pad1) -> /LED
- D157 pad 3: Net-(D156-Pad1) -> /LED
- D158 pad 1: Net-(D158-Pad1) -> /LED
- D158 pad 3: Net-(D157-Pad1) -> /LED
- D159 pad 1: Net-(D159-Pad1) -> /LED
- D159 pad 3: Net-(D158-Pad1) -> /LED
- D160 pad 1: RGBDOUT5 -> /LED
- D160 pad 3: Net-(D159-Pad1) -> /LED
- D161 pad 1: Net-(D161-Pad1) -> /LED
- D161 pad 3: RGBDOUT5 -> /LED
- D162 pad 1: Net-(D163-Pad3) -> /LED
- D162 pad 3: Net-(D161-Pad1) -> /LED
- D163 pad 1: Net-(D163-Pad1) -> /LED
- D163 pad 3: Net-(D163-Pad3) -> /LED
- D164 pad 1: Net-(D164-Pad1) -> /LED
- D164 pad 3: Net-(D163-Pad1) -> /LED
- D165 pad 1: Net-(D165-Pad1) -> /LED
- D165 pad 3: Net-(D164-Pad1) -> /LED
- D166 pad 1: Net-(D167-Pad3) -> /LED
- D166 pad 3: Net-(D165-Pad1) -> /LED
- D167 pad 1: Net-(D167-Pad1) -> /LED
- D167 pad 3: Net-(D167-Pad3) -> /LED
- D168 pad 1: Net-(D168-Pad1) -> /LED
- D168 pad 3: Net-(D167-Pad1) -> /LED
- D169 pad 1: Net-(D169-Pad1) -> /LED
- D169 pad 3: Net-(D168-Pad1) -> /LED
- D170 pad 1: RGBDOUT6 -> /LED
- D170 pad 3: Net-(D169-Pad1) -> /LED
- D171 pad 1: Net-(D171-Pad1) -> /LED
- D171 pad 3: RGBDOUT6 -> /LED
- D172 pad 1: Net-(D172-Pad1) -> /LED
- D172 pad 3: Net-(D171-Pad1) -> /LED
- D173 pad 1: Net-(D173-Pad1) -> /LED
- D173 pad 3: Net-(D172-Pad1) -> /LED
- D174 pad 1: Net-(D174-Pad1) -> /LED
- D174 pad 3: Net-(D173-Pad1) -> /LED
- D175 pad 1: Net-(D175-Pad1) -> /LED
- D175 pad 3: Net-(D174-Pad1) -> /LED
- D176 pad 1: Net-(D177-Pad3) -> /LED
- D176 pad 3: Net-(D175-Pad1) -> /LED
- D177 pad 1: Net-(D177-Pad1) -> /LED
- D177 pad 3: Net-(D177-Pad3) -> /LED
- D178 pad 1: Net-(D178-Pad1) -> /LED
- D178 pad 3: Net-(D177-Pad1) -> /LED
- D179 pad 1: Net-(D180-Pad3) -> /LED
- D179 pad 3: Net-(D178-Pad1) -> /LED
- D180 pad 1: RGBDOUT7 -> /LED
- D180 pad 3: Net-(D180-Pad3) -> /LED
- D181 pad 1: Net-(D181-Pad1) -> /LED
- D181 pad 3: RGBDOUT7 -> /LED
- D182 pad 1: Net-(D182-Pad1) -> /LED
- D182 pad 3: Net-(D181-Pad1) -> /LED
- D183 pad 1: Net-(D183-Pad1) -> /LED
- D183 pad 3: Net-(D182-Pad1) -> /LED
- D184 pad 1: Net-(D184-Pad1) -> /LED
- D184 pad 3: Net-(D183-Pad1) -> /LED
- D185 pad 1: Net-(D185-Pad1) -> /LED
- D185 pad 3: Net-(D184-Pad1) -> /LED
- D186 pad 1: Net-(D186-Pad1) -> /LED
- D186 pad 3: Net-(D185-Pad1) -> /LED
- D187 pad 1: Net-(D188-Pad3) -> /LED
- D187 pad 3: Net-(D186-Pad1) -> /LED
- D188 pad 1: Net-(D189-Pad3) -> /LED
- D188 pad 3: Net-(D188-Pad3) -> /LED
- D189 pad 1: Net-(D189-Pad1) -> /LED
- D189 pad 3: Net-(D189-Pad3) -> /LED
- D190 pad 1: RGBDOUT8 -> /LED
- D190 pad 3: Net-(D189-Pad1) -> /LED
- D191 pad 1: Net-(D191-Pad1) -> /LED
- D191 pad 3: RGBDOUT8 -> /LED
- D192 pad 1: Net-(D192-Pad1) -> /LED
- D192 pad 3: Net-(D191-Pad1) -> /LED
- D193 pad 1: Net-(D193-Pad1) -> /LED
- D193 pad 3: Net-(D192-Pad1) -> /LED
- D194 pad 1: Net-(D194-Pad1) -> /LED
- D194 pad 3: Net-(D193-Pad1) -> /LED
- D195 pad 1: Net-(D195-Pad1) -> /LED
- D195 pad 3: Net-(D194-Pad1) -> /LED
- D196 pad 1: Net-(D196-Pad1) -> /LED
- D196 pad 3: Net-(D195-Pad1) -> /LED
- D197 pad 1: Net-(D198-Pad3) -> /LED
- D197 pad 3: Net-(D196-Pad1) -> /LED
- D198 pad 1: Net-(D199-Pad3) -> /LED
- D198 pad 3: Net-(D198-Pad3) -> /LED
- D199 pad 1: Net-(D200-Pad3) -> /LED
- D199 pad 3: Net-(D199-Pad3) -> /LED
- D200 pad 1: unconnected-(D200-Pad1) -> /LED
- D200 pad 3: Net-(D200-Pad3) -> /LED
Routing:
- net /LED: track 0.00 -> 4127.8 mm, vias 0 -> 190
- net Net-(D159-Pad1): track 155.4 -> 0.00 mm, vias 2 -> 0
- net Net-(D171-Pad1): track 139.5 -> 0.00 mm, vias 2 -> 0
- net Net-(D165-Pad1): track 133.2 -> 0.00 mm, vias 4 -> 0
- net Net-(D139-Pad3): track 130.9 -> 0.00 mm, vias 2 -> 0
- net Net-(D178-Pad1): track 122.1 -> 0.00 mm, vias 2 -> 0
- net Net-(D117-Pad1): track 120.6 -> 0.00 mm, vias 2 -> 0
- net Net-(D153-Pad1): track 117.1 -> 0.00 mm, vias 2 -> 0
- net Net-(D111-Pad1): track 114.2 -> 0.00 mm, vias 2 -> 0
- net Net-(D148-Pad1): track 107.6 -> 0.00 mm, vias 2 -> 0
- net Net-(D144-Pad3): track 106.2 -> 0.00 mm, vias 2 -> 0
- net Net-(D132-Pad1): track 105.9 -> 0.00 mm, vias 2 -> 0
- net Net-(D123-Pad3): track 100.1 -> 0.00 mm, vias 2 -> 0
- net Net-(D127-Pad1): track 98.2 -> 0.00 mm, vias 2 -> 0
- net Net-(D193-Pad1): track 97.8 -> 0.00 mm, vias 2 -> 0
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
Commit message: led go brrrr
Routing:
- net GND: track 88.3 -> 4670.9 mm, vias 0 -> 23
- net +5V: track 400.5 -> 3562.8 mm, vias 1 -> 204
- net COL7: track 450.0 -> 451.9 mm
- net COL8: track 404.8 -> 406.6 mm
- net COL5: track 506.8 -> 508.6 mm
- net ROW0: track 407.0 -> 408.2 mm
- net /LED: track 4127.8 -> 4128.6 mm, vias 190 -> 192

Commit message: mcu
Parts:
- moved SW1 75.0 mm to (475.6, 187.0), turned to 180 degrees
- moved C6 61.4 mm to (464.6, 184.6), turned to -45 degrees
- moved Y1 59.6 mm to (466.8, 182.4), turned to 135 degrees
- moved C8 47.7 mm to (437.6, 186.0), turned to -135 degrees
- moved C5 44.6 mm to (468.9, 180.1), turned to 135 degrees
- moved R6 43.0 mm to (460.2, 188.8), turned to 135 degrees
- moved R4 40.1 mm to (435.6, 184.0), turned to -135 degrees
- moved R5 38.3 mm to (460.4, 166.2), turned to 45 degrees
- moved R3 35.2 mm to (433.6, 182.2), turned to -135 degrees
- moved C7 2.83 mm to (441.2, 185.6)
- moved C4 2.28 mm to (462.2, 186.8), turned to 135 degrees
Routing:
- net D+: track 2.92 -> 343.2 mm, vias 0 -> 3
- net D-: track 2.99 -> 340.3 mm, vias 0 -> 3
- net GND: track 4670.9 -> 4723.5 mm, vias 23 -> 24
- net Net-(R6-Pad2): track 0.00 -> 32.4 mm, vias 0 -> 2
- net +5V: track 3562.8 -> 3578.9 mm
- net Net-(C5-Pad1): track 0.00 -> 15.7 mm, vias 0 -> 2
- net Net-(R3-Pad1): track 0.00 -> 13.0 mm, vias 0 -> 2
- net Net-(C6-Pad1): track 0.00 -> 11.9 mm
- net Net-(R4-Pad1): track 0.00 -> 11.1 mm, vias 0 -> 2
- net Net-(C8-Pad1): track 0.00 -> 10.6 mm, vias 0 -> 2
- net Net-(R5-Pad1): track 0.00 -> 3.54 mm
