File: PCB/pcb.kicad_sch (KiCad schematic)
At the start: 324 parts, among them J1 USB_C_Receptacle_USB2.0, SW1 SW_Push, U1 AT90USB1286-AU, Y1 Crystal_GND24_Small

Commit message: change footprint
Parts:
- D1: Item (none) -> 1N4148W; LCSC (none) -> https://lcsc.com/product-detail/Switching-Diode_GOODWORK-1N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
Changed lines of the file:
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@@
     )
     (property "Name" "Esc" (id 4) (at 217.17 46.99 0))
+    (property "Item" "1N4148W" (id 5) (at 219.71 49.53 0)
+      (effects (font (size 1.27 1.27)) hide)
+    )
+    (property "LCSC" "https://lcsc.com/product-detail/Switching-Diode_GOODWORK-1N4148W_C909967.html" (id 6) (at 219.71 49.53 0)
+      (effects (font (size 1.27 1.27)) hide)
+    )
     (pin "1")
     (pin "2")

Commit message: switchj
Parts:
- C3: footprint Capacitor_SMD:C_0805_2012Metric -> led:switch_without_switch
- D1, D10, D100, D11, D12, D13, D14, D15, D16, D17, D18, D19, D2, D20, D21, D22, D23, D24, D25, D26, D27, D28, D29, D3, D30, D31, D32, D33, D34, D35, D36, D37, D38, D39, D4, D40, D41, D42, D43, D44, D45, D46, D47, D48, D49, D5, D50, D51, D52, D53, D54, D55, D56, D57, D58, D59, D6, D60, D61, D62, D63, D64, D65, D66, D67, D68, D69, D7, D70, D71, D72, D73, D74, D75, D76, D77, D78, D79, D8, D80, D81, D82, D83, D84, D85, D86, D87, D88, D89, D9, D90, D91, D92, D93, D94, D95, D96, D97, D98, D99: value (none) -> 1.25V@150mA; footprint (none) -> led:D_SOD-123
- SW1: footprint random-keyboard-parts:SKQG-1155865 -> led:switch_without_switch

Commit message: Revert "switchj"
This reverts commit d5a96ddcb071ce4a4afd099785118bfee5e594ee.
Parts:
- C3: footprint led:switch_without_switch -> Capacitor_SMD:C_0805_2012Metric
- D1, D10, D100, D11, D12, D13, D14, D15, D16, D17, D18, D19, D2, D20, D21, D22, D23, D24, D25, D26, D27, D28, D29, D3, D30, D31, D32, D33, D34, D35, D36, D37, D38, D39, D4, D40, D41, D42, D43, D44, D45, D46, D47, D48, D49, D5, D50, D51, D52, D53, D54, D55, D56, D57, D58, D59, D6, D60, D61, D62, D63, D64, D65, D66, D67, D68, D69, D7, D70, D71, D72, D73, D74, D75, D76, D77, D78, D79, D8, D80, D81, D82, D83, D84, D85, D86, D87, D88, D89, D9, D90, D91, D92, D93, D94, D95, D96, D97, D98, D99: value 1.25V@150mA -> (none); footprint led:D_SOD-123 -> (none)
- SW1: footprint led:switch_without_switch -> random-keyboard-parts:SKQG-1155865

Commit message: some silk
Parts:
- D1, D10, D100, D11, D12, D13, D14, D15, D16, D17, D18, D19, D2, D20, D21, D22, D23, D24, D25, D26, D27, D28, D29, D3, D30, D31, D32, D33, D34, D35, D36, D37, D38, D39, D4, D40, D41, D42, D43, D44, D45, D46, D47, D48, D49, D5, D50, D51, D52, D53, D54, D55, D56, D57, D58, D59, D6, D60, D61, D62, D63, D64, D65, D66, D67, D68, D69, D7, D70, D71, D72, D73, D74, D75, D76, D77, D78, D8, D80, D81, D82, D83, D84, D85, D86, D87, D88, D89, D9, D90, D91, D92, D93, D94, D95, D96, D97, D98, D99: value (none) -> 1.25V@150mA; footprint (none) -> led:D_SOD-123
- D79: Name Druck -> Print

Commit message: All Rows and Columns connected
Parts:
- D79: value (none) -> 1.25V@150mA; footprint (none) -> led:D_SOD-123
Connections:
- net COL0: now also U1.59 (PF2)
- net COL1: now also U1.60 (PF1)
- net COL10: now also U1.17 (PB7)
- net COL11: now also U1.18 (PE4)
- net COL12: now also U1.19 (PE5)
- net COL13: now also U1.25 (PD0)
- net COL14: now also U1.26 (PD1)
- net COL15: now also U1.27 (PD2)
- net COL16: now also U1.29 (PD4)
- net COL17: now also U1.31 (PD6)
- net COL2: now also U1.9 (PE3)
- net COL3: now also U1.10 (PB0)
- net COL4: now also U1.11 (PB1)
- net COL5: now also U1.12 (PB2)
- net COL6: now also U1.13 (PB3)
- net COL7: now also U1.14 (PB4)
- net COL8: now also U1.15 (PB5)
- net COL9: now also U1.16 (PB6)
- net ROW0: now also U1.30 (PD5)
- net ROW1: now also U1.2 (PE7)
- net ROW2: now also U1.28 (PD3)
- net ROW3: now also U1.1 (PE6)
- net ROW4: now also U1.61 (PF0)
- net ROW5: now also U1.32 (PD7)
Changed lines of the file:
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@@
     (effects (font (size 1.27 1.27)) (justify right bottom))
   )
+  (global_label "ROW5" (shape input) (at 182.88 125.73 0) (fields_autoplaced)
+    (effects (font (size 1.27 1.27)) (justify left))
+    (property "Intersheet References" "${INTERSHEET_REFS}" (id 0) (at 217.17 398.78 0)
+      (effects (font (size 1.27 1.27)) hide)
+    )
+  )
   (global_label "COL12" (shape input) (at 473.71 35.56 90) (fields_autoplaced)
     (effects (font (size 1.27 1.27)) (justify left))
@@
     )
   )
+  (global_label "COL13" (shape input) (at 182.88 107.95 0) (fields_autoplaced)
+    (effects (font (size 1.27 1.27)) (justify left))
+    (property "Intersheet References" "${INTERSHEET_REFS}" (id 0) (at 344.17 -210.82 0)
+      (effects (font (size 1.27 1.27)) hide)
+    )
+  )
   (global_label "COL0" (shape input) (at 229.87 35.56 90) (fields_autoplaced)
     (effects (font (size 1.27 1.27)) (justify left))
@@
     )
   )
+  (global_label "COL12" (shape input) (at 152.4 97.79 180) (fields_autoplaced)
+    (effects (font (size 1.27 1.27)) (justify right))
+    (property "Intersheet References" "${INTERSHEET_REFS}" (id 0) (at -8.89 396.24 0)
+      (effects (font (size 1.27 1.27)) hide)
+    )
+  )
+  (global_label "COL14" (shape input) (at 182.88 110.49 0) (fields_autoplaced)
+    (effects (font (size 1.27 1.27)) (justify left))
+    (property "Intersheet References" "${INTERSHEET_REFS}" (id 0) (at 344.17 -261.62 0)
+      (effects (font (size 1.27 1.27)) hide)
+    )
+  )
   (global_label "RGBDIN" (shape input) (at 38.1 185.42 180) (fields_autoplaced)
     (effects (font (size 1.27 1.27)) (justify right))
@@
     )
   )
+  (global_label "COL17" (shape input) (at 182.88 123.19 0) (fields_autoplaced)
+    (effects (font (size 1.27 1.27)) (justify left))
+    (property "Intersheet References" "${INTERSHEET_REFS}" (id 0) (at 344.17 -342.9 0)
+      (effects (font (size 1.27 1.27)) hide)
+    )
+  )
   (global_label "COL7" (shape input) (at 372.11 35.56 90) (fields_autoplaced)
     (effects (font (size 1.27 1.27)) (justify left))
@@
     )
   )
+  (global_label "COL16" (shape input) (at 182.88 118.11 0) (fields_autoplaced)
+    (effects (font (size 1.27 1.27)) (justify left))
+    (property "Intersheet References" "${INTERSHEET_REFS}" (id 0) (at 344.17 -307.34 0)
+      (effects (font (size 1.27 1.27)) hide)
+    )
+  )
+  (global_label "COL15" (shape input) (at 182.88 113.03 0) (fields_autoplaced)
+    (effects (font (size 1.27 1.27)) (justify left))
+    (property "Intersheet References" "${INTERSHEET_REFS}" (id 0) (at 344.17 -292.1 0)
+      (effects (font (size 1.27 1.27)) hide)
+    )
+  )
   (global_label "ROW3" (shape input) (at 209.55 109.22 180) (fields_autoplaced)
     (effects (font (size 1.27 1.27)) (justify right))
@@
     )
   )
+  (global_label "ROW0" (shape input) (at 182.88 120.65 0) (fields_autoplaced)
+    (effects (font (size 1.27 1.27)) (justify left))
+    (property "Intersheet References" "${INTERSHEET_REFS}" (id 0) (at 217.17 298.45 0)
+      (effects (font (size 1.27 1.27)) hide)
+    )
+  )
   (global_label "ROW5" (shape input) (at 209.55 147.32 180) (fields_autoplaced)
     (effects (font (size 1.27 1.27)) (justify right))
@@
     )
   )
+  (global_label "ROW1" (shape input) (at 152.4 102.87 180) (fields_autoplaced)
+    (effects (font (size 1.27 1.27)) (justify right))
+    (property "Intersheet References" "${INTERSHEET_REFS}" (id 0) (at 118.11 -93.98 0)
+      (effects (font (size 1.27 1.27)) hide)
+    )
+  )
   (global_label "COL14" (shape input) (at 547.37 35.56 90) (fields_autoplaced)
     (effects (font (size 1.27 1.27)) (justify left))
@@
     )
   )
+  (global_label "ROW2" (shape input) (at 182.88 115.57 0) (fields_autoplaced)
+    (effects (font (size 1.27 1.27)) (justify left))
+    (property "Intersheet References" "${INTERSHEET_REFS}" (id 0) (at 217.17 331.47 0)
+      (effects (font (size 1.27 1.27)) hide)
+    )
+  )
   (global_label "COL6" (shape input) (at 351.79 35.56 90) (fields_autoplaced)
     (effects (font (size 1.27 1.27)) (justify left))
@@
     )
   )
+  (global_label "COL7" (shape input) (at 182.88 72.39 0) (fields_autoplaced)
+    (effects (font (size 1.27 1.27)) (justify left))
+    (property "Intersheet References" "${INTERSHEET_REFS}" (id 0) (at 344.17 -124.46 0)
+      (effects (font (size 1.27 1.27)) hide)
+    )
+  )
   (global_label "COL1" (shape input) (at 250.19 35.56 90) (fields_autoplaced)
     (effects (font (size 1.27 1.27)) (justify left))
@@
     )
   )
+  (global_label "COL4" (shape input) (at 182.88 64.77 0) (fields_autoplaced)
+    (effects (font (size 1.27 1.27)) (justify left))
+    (property "Intersheet References" "${INTERSHEET_REFS}" (id 0) (at 344.17 -71.12 0)
+      (effects (font (size 1.27 1.27)) hide)
+    )
+  )
   (global_label "ROW4" (shape input) (at 209.55 128.27 180) (fields_autoplaced)
     (effects (font (size 1.27 1.27)) (justify right))
@@
     )
   )
+  (global_label "COL8" (shape input) (at 182.88 74.93 0) (fields_autoplaced)
+    (effects (font (size 1.27 1.27)) (justify left))
+    (property "Intersheet References" "${INTERSHEET_REFS}" (id 0) (at 344.17 -142.24 0)
+      (effects (font (size 1.27 1.27)) hide)
+    )
+  )
   (global_label "COL2" (shape input) (at 270.51 35.56 90) (fields_autoplaced)
     (effects (font (size 1.27 1.27)) (justify left))
@@
     )
   )
+  (global_label "COL1" (shape input) (at 152.4 110.49 180) (fields_autoplaced)
+    (effects (font (size 1.27 1.27)) (justify right))
+    (property "Intersheet References" "${INTERSHEET_REFS}" (id 0) (at -8.89 185.42 0)
+      (effects (font (size 1.27 1.27)) hide)
+    )
+  )
+  (global_label "COL10" (shape input) (at 182.88 80.01 0) (fields_autoplaced)
+    (effects (font (size 1.27 1.27)) (justify left))
+    (property "Intersheet References" "${INTERSHEET_REFS}" (id 0) (at 344.17 -177.8 0)
+      (effects (font (size 1.27 1.27)) hide)
+    )
+  )
+  (global_label "COL9" (shape input) (at 182.88 77.47 0) (fields_autoplaced)
+    (effects (font (size 1.27 1.27)) (justify left))
+    (property "Intersheet References" "${INTERSHEET_REFS}" (id 0) (at 344.17 -160.02 0)
+      (effects (font (size 1.27 1.27)) hide)
+    )
+  )
   (global_label "COL3" (shape input) (at 290.83 35.56 90) (fields_autoplaced)
     (effects (font (size 1.27 1.27)) (justify left))
@@
     )
   )
+  (global_label "ROW3" (shape input) (at 152.4 100.33 180) (fields_autoplaced)
+    (effects (font (size 1.27 1.27)) (justify right))
+    (property "Intersheet References" "${INTERSHEET_REFS}" (id 0) (at 118.11 -134.62 0)
+      (effects (font (size 1.27 1.27)) hide)
+    )
+  )
+  (global_label "COL0" (shape input) (at 152.4 113.03 180) (fields_autoplaced)
+    (effects (font (size 1.27 1.27)) (justify right))
+    (property "Intersheet References" "${INTERSHEET_REFS}" (id 0) (at -8.89 167.64 0)
+      (effects (font (size 1.27 1.27)) hide)
+    )
+  )
+  (global_label "COL3" (shape input) (at 182.88 62.23 0) (fields_autoplaced)
+    (effects (font (size 1.27 1.27)) (justify left))
+    (property "Intersheet References" "${INTERSHEET_REFS}" (id 0) (at 344.17 -53.34 0)
+      (effects (font (size 1.27 1.27)) hide)
+    )
+  )
   (global_label "COL9" (shape input) (at 412.75 35.56 90) (fields_autoplaced)
     (effects (font (size 1.27 1.27)) (justify left))
@@
     )
   )
+  (global_label "COL6" (shape input) (at 182.88 69.85 0) (fields_autoplaced)
+    (effects (font (size 1.27 1.27)) (justify left))
+    (property "Intersheet References" "${INTERSHEET_REFS}" (id 0) (at 344.17 -106.68 0)
+      (effects (font (size 1.27 1.27)) hide)
+    )
+  )
   (global_label "COL10" (shape input) (at 433.07 35.56 90) (fields_autoplaced)
     (effects (font (size 1.27 1.27)) (justify left))
@@
     )
   )
+  (global_label "ROW4" (shape input) (at 152.4 107.95 180) (fields_autoplaced)
+    (effects (font (size 1.27 1.27)) (justify right))
+    (property "Intersheet References" "${INTERSHEET_REFS}" (id 0) (at 118.11 -146.05 0)
+      (effects (font (size 1.27 1.27)) hide)
+    )
+  )
+  (global_label "COL11" (shape input) (at 152.4 95.25 180) (fields_autoplaced)
+    (effects (font (size 1.27 1.27)) (justify right))
+    (property "Intersheet References" "${INTERSHEET_REFS}" (id 0) (at -8.89 373.38 0)
+      (effects (font (size 1.27 1.27)) hide)
+    )
+  )
   (global_label "COL8" (shape input) (at 392.43 35.56 90) (fields_autoplaced)
     (effects (font (size 1.27 1.27)) (justify left))
@@
     )
   )
+  (global_label "COL5" (shape input) (at 182.88 67.31 0) (fields_autoplaced)
+    (effects (font (size 1.27 1.27)) (justify left))
+    (property "Intersheet References" "${INTERSHEET_REFS}" (id 0) (at 344.17 -88.9 0)
+      (effects (font (size 1.27 1.27)) hide)
+    )
+  )
   (global_label "COL16" (shape input) (at 600.71 35.56 90) (fields_autoplaced)
     (effects (font (size 1.27 1.27)) (justify left))
@@
     )
   )
+  (global_label "COL2" (shape input) (at 152.4 92.71 180) (fields_autoplaced)
+    (effects (font (size 1.27 1.27)) (justify right))
+    (property "Intersheet References" "${INTERSHEET_REFS}" (id 0) (at -8.89 187.96 0)
+      (effects (font (size 1.27 1.27)) hide)
+    )
+  )
   (symbol (lib_id "pcb-rescue:AT90USB1286-AU-MCU_Microchip_AVR") (at 167.64 82.55 0) (unit 1)
     (in_bom yes) (on_board yes)
@@
       (effects (font (size 1.27 1.27)) (justify right))
     )
-    (property "Value" "" (id 1) (at 534.67 30.48 0)
+    (property "Value" "1.25V@150mA" (id 1) (at 534.67 30.48 0)
       (effects (font (size 1.27 1.27)) (justify right))
     )
-    (property "Footprint" "" (id 2) (at 537.21 49.53 90)
+    (property "Footprint" "led:D_SOD-123" (id 2) (at 537.21 49.53 90)
       (effects (font (size 1.27 1.27)) hide)
     )

Commit message: LED Data Bus connected
Connections:
- net RGBDIN: now also U1.51 (PA0)
Changed lines of the file:
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@@
+    )
+  )
+  (global_label "RGBDIN" (shape input) (at 182.88 39.37 0) (fields_autoplaced)
+    (effects (font (size 1.27 1.27)) (justify left))
+    (property "Intersheet References" "${INTERSHEET_REFS}" (id 0) (at 192.2194 39.4494 0)
+      (effects (font (size 1.27 1.27)) (justify left) hide)
     )
   )

Commit message: Reset Switch Footprint Updated
Parts:
- D21: footprint led:D_SOD-123 -> (none)
- SW1: footprint random-keyboard-parts:SKQG-1155865 -> (none)
Changed lines of the file:
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@@
     (property "Reference" "SW1" (id 0) (at 142.24 32.131 0))
     (property "Value" "SW_Push" (id 1) (at 142.24 34.4424 0))
-    (property "Footprint" "random-keyboard-parts:SKQG-1155865" (id 2) (at 142.24 34.29 0)
+    (property "Footprint" "" (id 2) (at 142.24 34.29 0)
       (effects (font (size 1.27 1.27)) hide)
     )
@@
       (effects (font (size 1.27 1.27)) (justify right))
     )
-    (property "Footprint" "led:D_SOD-123" (id 2) (at 280.67 106.68 90)
+    (property "Footprint" "" (id 2) (at 280.67 106.68 90)
       (effects (font (size 1.27 1.27)) hide)
     )
@@
     )
     (path "/00000000-0000-0000-0000-00006236ed86"
-      (reference "D21") (unit 1) (value "1.25V@150mA") (footprint "led:D_SOD-123")
+      (reference "D21") (unit 1) (value "1.25V@150mA") (footprint "led:switch_without_switch")
     )
     (path "/00000000-0000-0000-0000-00006236ed93"
@@
     )
     (path "/00000000-0000-0000-0000-000062265bdd"
-      (reference "SW1") (unit 1) (value "SW_Push") (footprint "random-keyboard-parts:SKQG-1155865")
+      (reference "SW1") (unit 1) (value "SW_Push") (footprint "led:switch_without_switch")
     )
     (path "/00000000-0000-0000-0000-00006223ede6"

Commit message: Silkscreen Legends updated
Parts:
- D10: Name < -> \
- D57: Name Ö -> ;
- D61: Name ß -> -
- D62: Name Ü -> [
- D63: Name Ä -> '
- D64: Name - -> /
- D67: Name ´ -> =
- D68: Name + -> ]
Changed lines of the file:
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@@
       (effects (font (size 1.27 1.27)) hide)
     )
-    (property "Name" "<" (id 4) (at 237.49 123.19 0))
+    (property "Name" "\\" (id 4) (at 237.49 123.19 0))
     (pin "1")
     (pin "2")
@@
       (effects (font (size 1.27 1.27)) hide)
     )
-    (property "Name" "ß" (id 4) (at 440.69 66.04 0))
+    (property "Name" "-" (id 4) (at 440.69 66.04 0))
     (pin "1")
     (pin "2")
@@
       (effects (font (size 1.27 1.27)) hide)
     )
-    (property "Name" "Ü" (id 4) (at 440.69 85.09 0))
+    (property "Name" "[" (id 4) (at 440.69 85.09 0))
     (pin "1")
     (pin "2")
@@
       (effects (font (size 1.27 1.27)) hide)
     )
-    (property "Name" "Ö" (id 4) (at 420.37 104.14 0))
+    (property "Name" ";" (id 4) (at 420.37 104.14 0))
     (pin "1")
     (pin "2")
@@
       (effects (font (size 1.27 1.27)) hide)
     )
-    (property "Name" "Ä" (id 4) (at 440.69 104.14 0))
+    (property "Name" "'" (id 4) (at 440.69 104.14 0))
     (pin "1")
     (pin "2")
@@
       (effects (font (size 1.27 1.27)) hide)
     )
-    (property "Name" "-" (id 4) (at 440.69 123.19 0))
+    (property "Name" "/" (id 4) (at 440.69 123.19 0))
     (pin "1")
     (pin "2")
@@
       (effects (font (size 1.27 1.27)) hide)
     )
-    (property "Name" "´" (id 4) (at 461.01 66.04 0))
+    (property "Name" "=" (id 4) (at 461.01 66.04 0))
     (pin "1")
     (pin "2")
@@
       (effects (font (size 1.27 1.27)) hide)
     )
-    (property "Name" "+" (id 4) (at 461.01 85.09 0))
+    (property "Name" "]" (id 4) (at 461.01 85.09 0))
     (pin "1")
     (pin "2")
@@
     )
     (path "/00000000-0000-0000-0000-00006236ed86"
-      (reference "D21") (unit 1) (value "1.25V@150mA") (footprint "led:switch_without_switch")
+      (reference "D21") (unit 1) (value "1.25V@150mA") (footprint "led:D_SOD-123")
     )
     (path "/00000000-0000-0000-0000-00006236ed93"
