File: MacroBoard/MacroBoard.kicad_pcb (KiCad board)
At the start: 2 copper layers, 3.9 x 3.7 mm, 80 parts, among them J1 USB_C_Receptacle_USB2.0, SW1 SW_Push, U1 AT90USB1286-AU, Y1 Crystal_GND24_Small

Commit message: macro board
Parts:
- added C10: 100nF, led:led_capacitor, B.Cu at (74.8, 90.3)
- added C11: 100nF, led:led_capacitor, B.Cu at (74.7, 109.3)
- added C12: 100nF, led:led_capacitor, B.Cu at (74.7, 128.4)
- added C13: 100nF, led:led_capacitor, B.Cu at (93.8, 71.2)
- added C14: 100nF, led:led_capacitor, B.Cu at (93.7, 90.3)
- added C15: 100nF, led:led_capacitor, B.Cu at (93.8, 109.3)
- added C16: 100nF, led:led_capacitor, B.Cu at (93.8, 128.4)
- added C17: 100nF, led:led_capacitor, B.Cu at (112.8, 71.2)
- added C18: 100nF, led:led_capacitor, B.Cu at (112.9, 90.3)
- added C19: 100nF, led:led_capacitor, B.Cu at (112.9, 109.3)
- added C20: 100nF, led:led_capacitor, B.Cu at (112.8, 128.4)
- added C21: 100nF, led:led_capacitor, B.Cu at (131.8, 71.2)
- added C22: 100nF, led:led_capacitor, B.Cu at (131.9, 90.3)
- added C23: 100nF, led:led_capacitor, B.Cu at (131.9, 109.3)
- added C24: 100nF, led:led_capacitor, B.Cu at (131.9, 128.4)
- added C25: 100nF, led:led_capacitor, B.Cu at (150.9, 71.2)
- added C26: 100nF, led:led_capacitor, B.Cu at (150.9, 90.3)
- added C27: 100nF, led:led_capacitor, B.Cu at (151.0, 109.3)
- added C28: 100nF, led:led_capacitor, B.Cu at (150.9, 128.4)
- added C9: 100nF, led:led_capacitor, B.Cu at (74.6, 71.2)
- moved D13 4.05 mm to (129.4, 65.9), turned to 0 degrees
- moved D14 4.05 mm to (129.4, 84.9), turned to 0 degrees
- moved D15 4.05 mm to (129.4, 104.0), turned to 0 degrees
- moved D16 4.05 mm to (129.4, 123.0), turned to 0 degrees
- moved D10 4.05 mm to (110.3, 84.9), turned to 0 degrees
- moved D11 4.05 mm to (110.3, 104.0), turned to 0 degrees
- moved D12 4.05 mm to (110.3, 123.0), turned to 0 degrees
- moved D5 4.05 mm to (91.3, 65.9), turned to 0 degrees
- moved D6 4.05 mm to (91.3, 84.9), turned to 0 degrees
- moved D7 4.05 mm to (91.3, 104.0), turned to 0 degrees
- moved D9 4.05 mm to (110.3, 65.9), turned to 0 degrees
- moved D17 4.05 mm to (148.4, 65.9), turned to 0 degrees
- moved D18 4.05 mm to (148.4, 84.9), turned to 0 degrees
- moved D19 4.05 mm to (148.4, 104.0), turned to 0 degrees
- moved D20 4.05 mm to (148.4, 123.0), turned to 0 degrees
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Routing:
- net +5V: track 0.00 -> 384.6 mm
- net COL4: track 37.2 -> 259.9 mm, vias 0 -> 2
- net COL3: track 35.4 -> 237.2 mm, vias 0 -> 2
- net COL2: track 37.2 -> 217.8 mm, vias 0 -> 2
- net COL1: track 37.2 -> 196.8 mm, vias 0 -> 2
- net COL0: track 37.2 -> 175.7 mm, vias 0 -> 2
- net Net-(D22-Pad3): track 0.00 -> 111.9 mm, vias 0 -> 2
- net Net-(D24-Pad3): track 0.00 -> 111.9 mm, vias 0 -> 2
- net Net-(D23-Pad3): track 0.00 -> 111.9 mm, vias 0 -> 2
- net Net-(D20-Pad2): track 14.2 -> 94.6 mm
- net ROW0: track 0.00 -> 78.7 mm
- net ROW3: track 0.00 -> 78.4 mm
- net ROW2: track 0.00 -> 78.4 mm
- net ROW1: track 0.00 -> 78.4 mm
- net Net-(D19-Pad2): track 14.2 -> 75.4 mm
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
Commit message: makro board
Parts:
- C1, C2, C3, C4, C5, C6, C7, C8, F1, FB1, J1, R1, R2, R3, R4, R5, R6, U1, Y1: moved to B.Cu
- SW1: footprint random-keyboard-parts:SKQG-1155865 -> led:switch_without_switch; moved to B.Cu
- moved R1 68.4 mm to (77.7, 42.7)
- moved C6 60.2 mm to (162.6, 33.5), turned to 45 degrees
- moved R4 59.0 mm to (91.4, 46.9), turned to -135 degrees
- moved C1 54.8 mm to (76.7, 40.2), turned to 180 degrees
- moved F1 52.8 mm to (84.7, 40.6), turned to 90 degrees
- moved R5 49.7 mm to (98.1, 49.8), turned to -135 degrees
- moved FB1 47.8 mm to (88.0, 42.0), turned to 180 degrees
- moved R3 47.5 mm to (93.2, 48.6), turned to -135 degrees
- moved Y1 46.9 mm to (166.0, 34.6), turned to -135 degrees
- moved C5 36.3 mm to (167.1, 38.0), turned to -135 degrees
- moved R2 33.2 mm to (82.8, 44.4), turned to 180 degrees
- moved R6 30.9 mm to (122.2, 49.4)
- moved C7 23.9 mm to (97.7, 36.9), turned to 135 degrees
- moved C8 19.9 mm to (129.3, 39.5), turned to -45 degrees
- moved U1 19.9 mm to (108.7, 42.9), turned to -135 degrees
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Connections:
- U1 pad 29: unconnected-(U1-Pad29) -> ROW3
- U1 pad 30: unconnected-(U1-Pad30) -> ROW2
- U1 pad 31: unconnected-(U1-Pad31) -> ROW1
- U1 pad 32: unconnected-(U1-Pad32) -> ROW0
- U1 pad 33: unconnected-(U1-Pad33) -> COL0
- U1 pad 34: unconnected-(U1-Pad34) -> COL1
- U1 pad 35: unconnected-(U1-Pad35) -> COL2
- U1 pad 36: unconnected-(U1-Pad36) -> COL3
- U1 pad 37: unconnected-(U1-Pad37) -> COL4
Routing:
- net ROW3: track 78.4 -> 223.6 mm
- net ROW2: track 78.4 -> 204.2 mm
- net ROW1: track 78.4 -> 184.6 mm
- net ROW0: track 78.7 -> 165.2 mm
- net Net-(D20-Pad2): track 94.6 -> 12.7 mm
- net +5V: track 384.6 -> 462.5 mm
- net Net-(C5-Pad1): track 0.00 -> 69.1 mm
- net Net-(D19-Pad2): track 75.4 -> 12.7 mm
- net Net-(C6-Pad1): track 0.00 -> 62.6 mm
- net Net-(D18-Pad2): track 56.1 -> 12.7 mm
- net Net-(R4-Pad1): track 0.00 -> 30.3 mm, vias 0 -> 2
- net GND: track 0.00 -> 28.6 mm, vias 0 -> 47
- net D-: track 0.00 -> 28.0 mm
- net Net-(R3-Pad1): track 0.00 -> 27.4 mm, vias 0 -> 2
- net D+: track 0.00 -> 25.8 mm
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- added copper zone on B.Cu, net GND
- added copper zone on F.Cu, net GND
Other:
- board size 3.9 x 3.7 mm -> 103.3 x 105.9 mm
