File: Backplate/plate.kicad_pcb (KiCad board)
At the start: 2 copper layers, 400 x 123.8 mm, 0 parts

Commit message: Added Plate Gaskets
Diom Logo on Plate
Other:
- board size 400 x 123.8 mm -> 419.8 x 143.8 mm

Commit message: Gerber Files
Parts:
- added REF**: MountingHole_2.2mm_M2, MountingHole:MountingHole_2.2mm_M2, F.Cu at (350.3, 78.5)
- added REF**: MountingHole_2.2mm_M2, MountingHole:MountingHole_2.2mm_M2, F.Cu at (370.1, 78.5)
- added REF**: MountingHole_2.2mm_M2, MountingHole:MountingHole_2.2mm_M2, F.Cu at (3.81, 146.9)
- added REF**: MountingHole_2.2mm_M2, MountingHole:MountingHole_2.2mm_M2, F.Cu at (60.2, 78.5)
- added REF**: MountingHole_2.2mm_M2, MountingHole:MountingHole_2.2mm_M2, F.Cu at (370.1, 215.3)
- added REF**: MountingHole_2.2mm_M2, MountingHole:MountingHole_2.2mm_M2, F.Cu at (170.1, 215.3)
- added REF**: MountingHole_2.2mm_M2, MountingHole:MountingHole_2.2mm_M2, F.Cu at (160.2, 78.5)
- added REF**: MountingHole_2.2mm_M2, MountingHole:MountingHole_2.2mm_M2, F.Cu at (160.2, 215.3)
- added REF**: MountingHole_2.2mm_M2, MountingHole:MountingHole_2.2mm_M2, F.Cu at (60.2, 215.3)
- added REF**: MountingHole_2.2mm_M2, MountingHole:MountingHole_2.2mm_M2, F.Cu at (350.3, 215.3)
- added REF**: MountingHole_2.2mm_M2, MountingHole:MountingHole_2.2mm_M2, F.Cu at (150.3, 78.5)
- added REF**: MountingHole_2.2mm_M2, MountingHole:MountingHole_2.2mm_M2, F.Cu at (360.2, 78.5)
- added REF**: MountingHole_2.2mm_M2, MountingHole:MountingHole_2.2mm_M2, F.Cu at (416.6, 146.9)
- added REF**: MountingHole_2.2mm_M2, MountingHole:MountingHole_2.2mm_M2, F.Cu at (3.81, 137.0)
- added REF**: MountingHole_2.2mm_M2, MountingHole:MountingHole_2.2mm_M2, F.Cu at (70.1, 215.3)
- added REF**: MountingHole_2.2mm_M2, MountingHole:MountingHole_2.2mm_M2, F.Cu at (416.6, 137.0)
- added REF**: MountingHole_2.2mm_M2, MountingHole:MountingHole_2.2mm_M2, F.Cu at (270.1, 215.3)
- added REF**: MountingHole_2.2mm_M2, MountingHole:MountingHole_2.2mm_M2, F.Cu at (70.1, 78.5)
- added REF**: MountingHole_2.2mm_M2, MountingHole:MountingHole_2.2mm_M2, F.Cu at (270.1, 78.5)
- added REF**: MountingHole_2.2mm_M2, MountingHole:MountingHole_2.2mm_M2, F.Cu at (260.2, 215.3)
- added REF**: MountingHole_2.2mm_M2, MountingHole:MountingHole_2.2mm_M2, F.Cu at (170.1, 78.5)
- added REF**: MountingHole_2.2mm_M2, MountingHole:MountingHole_2.2mm_M2, F.Cu at (150.3, 215.3)
- added REF**: MountingHole_2.2mm_M2, MountingHole:MountingHole_2.2mm_M2, F.Cu at (50.3, 215.3)
- added REF**: MountingHole_2.2mm_M2, MountingHole:MountingHole_2.2mm_M2, F.Cu at (416.6, 156.8)
- added REF**: MountingHole_2.2mm_M2, MountingHole:MountingHole_2.2mm_M2, F.Cu at (360.2, 215.3)
- added REF**: MountingHole_2.2mm_M2, MountingHole:MountingHole_2.2mm_M2, F.Cu at (50.3, 78.5)
- added REF**: MountingHole_2.2mm_M2, MountingHole:MountingHole_2.2mm_M2, F.Cu at (250.3, 215.3)
- added REF**: MountingHole_2.2mm_M2, MountingHole:MountingHole_2.2mm_M2, F.Cu at (260.2, 78.5)
- added REF**: MountingHole_2.2mm_M2, MountingHole:MountingHole_2.2mm_M2, F.Cu at (250.3, 78.5)
- added REF**: MountingHole_2.2mm_M2, MountingHole:MountingHole_2.2mm_M2, F.Cu at (3.81, 156.8)
Other:
- outline, holes or cut-outs redrawn

Commit message: production and CAD preparations
Parts:
- removed REF** (x30): MountingHole_2.2mm_M2, MountingHole:MountingHole_2.2mm_M2
- added H1: MountingHole, Holes:MountingHoleM2, F.Cu at (416.6, 156.8)
- added H10: MountingHole, Holes:MountingHoleM2, F.Cu at (260.2, 215.3)
- added H11: MountingHole, Holes:MountingHoleM2, F.Cu at (360.2, 215.3)
- added H12: MountingHole, Holes:MountingHoleM2, F.Cu at (170.1, 215.3)
- added H13: MountingHole, Holes:MountingHoleM2, F.Cu at (3.81, 146.9)
- added H14: MountingHole, Holes:MountingHoleM2, F.Cu at (3.81, 156.8)
- added H15: MountingHole, Holes:MountingHoleM2, F.Cu at (160.2, 78.5)
- added H16: MountingHole, Holes:MountingHoleM2, F.Cu at (70.1, 78.5)
- added H17: MountingHole, Holes:MountingHoleM2, F.Cu at (270.1, 215.3)
- added H18: MountingHole, Holes:MountingHoleM2, F.Cu at (350.3, 78.5)
- added H19: MountingHole, Holes:MountingHoleM2, F.Cu at (250.3, 215.3)
- added H2: MountingHole, Holes:MountingHoleM2, F.Cu at (350.3, 215.3)
- added H20: MountingHole, Holes:MountingHoleM2, F.Cu at (170.1, 78.5)
- added H21: MountingHole, Holes:MountingHoleM2, F.Cu at (250.3, 78.5)
- added H22: MountingHole, Holes:MountingHoleM2, F.Cu at (70.1, 215.3)
- added H23: MountingHole, Holes:MountingHoleM2, F.Cu at (370.1, 78.5)
- added H24: MountingHole, Holes:MountingHoleM2, F.Cu at (416.6, 137.0)
- added H25: MountingHole, Holes:MountingHoleM2, F.Cu at (60.2, 78.5)
- added H26: MountingHole, Holes:MountingHoleM2, F.Cu at (50.3, 215.3)
- added H27: MountingHole, Holes:MountingHoleM2, F.Cu at (3.81, 137.1)
- added H28: MountingHole, Holes:MountingHoleM2, F.Cu at (416.6, 146.9)
- added H29: MountingHole, Holes:MountingHoleM2, F.Cu at (50.3, 78.5)
- added H3: MountingHole, Holes:MountingHoleM2, F.Cu at (360.2, 78.5)
- added H30: MountingHole, Holes:MountingHoleM2, F.Cu at (150.3, 215.3)
- added H4: MountingHole, Holes:MountingHoleM2, F.Cu at (370.1, 215.3)
- added H5: MountingHole, Holes:MountingHoleM2, F.Cu at (270.1, 78.5)
- added H6: MountingHole, Holes:MountingHoleM2, F.Cu at (60.2, 215.3)
- added H7: MountingHole, Holes:MountingHoleM2, F.Cu at (260.2, 78.5)
- added H8: MountingHole, Holes:MountingHoleM2, F.Cu at (160.2, 215.3)
- added H9: MountingHole, Holes:MountingHoleM2, F.Cu at (150.3, 78.5)
Other:
- outline, holes or cut-outs redrawn
